File: 01_Flightcontroller/Schematic/FC_WITHMPU6000/Flightcontroller.brd (EAGLE design)
At the start: 63.5 x 63.2 mm, 100 parts, among them Y1 8MHz, Y2 16MHz

Commit message: Umdrehen SD Karte
Parts:
- moved SD_CARD 0.28 mm to (18.0, 48.8), turned to 180 degrees
Routing:
- net GND: track 651.0 -> 709.4 mm, vias 43 -> 56
- net SD1_D0: track 91.9 -> 81.5 mm
- net VCC: track 317.4 -> 327.7 mm
- net SD1_CMD: track 44.3 -> 52.9 mm, vias 5 -> 7
- net SD1_CK: track 68.0 -> 67.1 mm
