File: 01_Flightcontroller/Schematic/FC_WITHICM-20689_rework/SHARKSKYFC.sch (EAGLE design)
At the start: 88 parts, among them IC1 FT232RL, IC2 BMP280, J1 2908-05WB-MG, U1 STM32F7X2RXT, U2 LM3940IMPX-3.3/NOPB, U3 ICM-20689, U4 ATMEGA328P_TQFP, Y1 8MHz, Y2 8MHz

Commit message: route new brd
Connections:
- removed net N$15: LED_1.C, LED_2.C, LED_3.C, ON.C
- net GND: now also LED_1.C, LED_2.C, LED_3.C, ON.C
Changed lines of the file:
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@@
 </variantdefs>
 <classes>
-<class number="0" name="default" width="0" drill="0">
+<class number="0" name="default" width="0.3048" drill="0">
 </class>
 </classes>
@@
 <part name="SUPPLY82" library="supply2" library_urn="urn:adsk.eagle:library:372" deviceset="GND" device=""/>
 <part name="SUPPLY83" library="SparkFun-PowerSymbols" library_urn="urn:adsk.eagle:library:530" deviceset="VCC_1" device=""/>
+<part name="SUPPLY78" library="supply2" library_urn="urn:adsk.eagle:library:372" deviceset="GND" device=""/>
 </parts>
 <sheets>
@@
 <instance part="SUPPLY83" gate="G$2" x="-368.3" y="111.76" smashed="yes" grouprefs="CONNECTORS">
 <attribute name="VALUE" x="-368.3" y="114.554" size="1.778" layer="96" align="bottom-center"/>
+</instance>
+<instance part="SUPPLY78" gate="GND" x="-312.42" y="40.64" smashed="yes">
+<attribute name="VALUE" x="-314.325" y="37.465" size="1.778" layer="96"/>
 </instance>
 </instances>
@@
 <wire x1="-368.3" y1="99.06" x2="-368.3" y2="96.52" width="0.1524" layer="91" grouprefs="CONNECTORS"/>
 </segment>
+<segment>
+<pinref part="LED_1" gate="G$1" pin="C"/>
+<wire x1="-322.58" y1="48.26" x2="-322.58" y2="45.72" width="0.1524" layer="91" grouprefs="CONNECTORS"/>
+<wire x1="-322.58" y1="45.72" x2="-314.96" y2="45.72" width="0.1524" layer="91" grouprefs="CONNECTORS"/>
+<pinref part="ON" gate="G$1" pin="C"/>
+<wire x1="-314.96" y1="45.72" x2="-312.42" y2="45.72" width="0.1524" layer="91" grouprefs="CONNECTORS"/>
+<wire x1="-312.42" y1="45.72" x2="-307.34" y2="45.72" width="0.1524" layer="91" grouprefs="CONNECTORS"/>
+<wire x1="-307.34" y1="45.72" x2="-299.72" y2="45.72" width="0.1524" layer="91" grouprefs="CONNECTORS"/>
+<wire x1="-299.72" y1="45.72" x2="-299.72" y2="48.26" width="0.1524" layer="91" grouprefs="CONNECTORS"/>
+<pinref part="LED_2" gate="G$1" pin="C"/>
+<wire x1="-314.96" y1="48.26" x2="-314.96" y2="45.72" width="0.1524" layer="91" grouprefs="CONNECTORS"/>
+<junction x="-314.96" y="45.72" grouprefs="CONNECTORS"/>
+<pinref part="LED_3" gate="G$1" pin="C"/>
+<wire x1="-307.34" y1="48.26" x2="-307.34" y2="45.72" width="0.1524" layer="91" grouprefs="CONNECTORS"/>
+<junction x="-307.34" y="45.72" grouprefs="CONNECTORS"/>
+<pinref part="SUPPLY78" gate="GND" pin="GND"/>
+<wire x1="-312.42" y1="43.18" x2="-312.42" y2="45.72" width="0.1524" layer="91"/>
+<junction x="-312.42" y="45.72"/>
+</segment>
 </net>
 <net name="VCC_1" class="0">
@@
 </segment>
 </net>
-<net name="N$15" class="0">
-<segment>
-<pinref part="LED_1" gate="G$1" pin="C"/>
-<wire x1="-322.58" y1="48.26" x2="-322.58" y2="45.72" width="0.1524" layer="91" grouprefs="CONNECTORS"/>
-<wire x1="-322.58" y1="45.72" x2="-314.96" y2="45.72" width="0.1524" layer="91" grouprefs="CONNECTORS"/>
-<pinref part="ON" gate="G$1" pin="C"/>
-<wire x1="-314.96" y1="45.72" x2="-307.34" y2="45.72" width="0.1524" layer="91" grouprefs="CONNECTORS"/>
-<wire x1="-307.34" y1="45.72" x2="-299.72" y2="45.72" width="0.1524" layer="91" grouprefs="CONNECTORS"/>
-<wire x1="-299.72" y1="45.72" x2="-299.72" y2="48.26" width="0.1524" layer="91" grouprefs="CONNECTORS"/>
-<pinref part="LED_2" gate="G$1" pin="C"/>
-<wire x1="-314.96" y1="48.26" x2="-314.96" y2="45.72" width="0.1524" layer="91" grouprefs="CONNECTORS"/>
-<junction x="-314.96" y="45.72" grouprefs="CONNECTORS"/>
-<pinref part="LED_3" gate="G$1" pin="C"/>
-<wire x1="-307.34" y1="48.26" x2="-307.34" y2="45.72" width="0.1524" layer="91" grouprefs="CONNECTORS"/>
-<junction x="-307.34" y="45.72" grouprefs="CONNECTORS"/>
-</segment>
-</net>
