File: 01_Flightcontroller/Schematic/FC_WITHICM-20689_rework/SHARKSKYFC.brd (EAGLE design)
At the start: 56.5 x 55.9 mm, 88 parts, among them IC1 FT232RL, IC2 BMP280, J1 2908-05WB-MG, U1 STM32F7X2RXT, U2 LM3940IMPX-3.3/NOPB, U3 ICM-20689, U4 ATMEGA328P_TQFP, Y1 8MHz, Y2 8MHz

Commit message: route new brd
Connections:
- removed net N$15: LED_1.C, LED_2.C, LED_3.C, ON.C
- net GND: now also LED_1.C, LED_2.C, LED_3.C, ON.C
Routing:
- net GND: track 148.0 -> 284.1 mm, vias 12 -> 23
- net VCC_2: track 54.3 -> 181.2 mm, vias 4 -> 9
- net VCC_1: track 93.1 -> 118.4 mm, vias 5 -> 7
- net RST: track 175.6 -> 176.9 mm

Commit message: more wiring 9 airwire left
Parts:
- moved C32 3.24 mm to (57.9, 55.4)
- moved C9 0.89 mm to (47.2, 79.5)
- moved Y1 0.89 mm to (49.1, 75.6)
- moved C4 0.77 mm to (37.2, 70.1)
- moved C23 0.25 mm to (61.5, 70.2)
Routing:
- net VCC_1: track 118.4 -> 177.2 mm, vias 7 -> 10
- net GND: track 284.1 -> 318.5 mm, vias 23 -> 27
- net CELL_3: track 23.2 -> 25.2 mm
- net RNG_ADC: track 44.0 -> 45.9 mm, vias 0 -> 2
- net VCC_2: track 181.2 -> 182.6 mm
- net IMU_MISO: track 16.1 -> 17.3 mm
- net USBOSD_TX: track 66.8 -> 67.6 mm
- net N$49: track 7.46 -> 8.15 mm
- net LED_2: track 67.3 -> 67.8 mm
- net LED_3: track 69.5 -> 70.0 mm
- net GIMBAL_Z: track 93.6 -> 94.0 mm, vias 7 -> 5
- net SWCLK: track 36.7 -> 36.8 mm, vias 1 -> 3
Other:
- board size 56.5 x 55.9 mm -> 56.5 x 56.6 mm
